File: pcb/fanned.kicad_pcb (KiCad board)
At the start: 4 copper layers, 46 x 86.4 mm, 79 parts, among them J1 USB4105-GF-A, J2 S2B-PH-SM4-TB, J3 FH12-40S-0.5SH(55), J4 SWD (BL652), J5 Console, Q1 DMG2302U, Q2 DMG2305UX, SW1 PTS810, SW2 PTS810, SW3 PTS810, SW4 SKRTLAE010, SW5 SKRTLAE010, U1 ESP32-S3-WROOM-1-N16R8, U2 BL652-SA-01, U3 MAX-M10S, U4 LTR-303ALS-01, U5 AP7361C-33E, U6 MCP73831-2, U7 MAX98357A, U8 BMP581

Commit message: pcb: v0.2 board fully routed - DRC 0 errors, 0 unconnected (5 intentional warnings); refs on fab layer, lib tables; cad: rotated key switches, board_fit OK on the routed board
Parts:
- AE1: footprint Taoglas_DSGP.1575.12.4.A.02_12x12mm -> OpenCycle:Taoglas_DSGP.1575.12.4.A.02_12x12mm
- C1, C12: footprint C_0805_2012Metric -> Capacitor_SMD:C_0805_2012Metric
- C10, C13, C17, C19, C2, C20, C3, C5, C7, C8: footprint C_0402_1005Metric -> Capacitor_SMD:C_0402_1005Metric
- C11, C14, C15, C16, C18, C4, C6, C9: footprint C_0603_1608Metric -> Capacitor_SMD:C_0603_1608Metric
- D1: footprint LED_0603_1608Metric -> LED_SMD:LED_0603_1608Metric
- D2: footprint SOT-23-6 -> Package_TO_SOT_SMD:SOT-23-6
- FID1, FID2, FID3, FID4, FID5, FID6: footprint Fiducial_0.75mm_Mask1.5mm -> Fiducial:Fiducial_0.75mm_Mask1.5mm
- H1, H2, H3, H4: footprint MountingHole_2.2mm_M2_Pad_Via -> MountingHole:MountingHole_2.2mm_M2_Pad_Via
- J1: footprint USB_C_Receptacle_GCT_USB4105-xx-A_16P_TopMnt_Horizontal -> Connector_USB:USB_C_Receptacle_GCT_USB4105-xx-A_16P_TopMnt_Horizontal
- J2: footprint JST_PH_S2B-PH-SM4-TB_1x02-1MP_P2.00mm_Horizontal -> Connector_JST:JST_PH_S2B-PH-SM4-TB_1x02-1MP_P2.00mm_Horizontal
- J3: footprint Hirose_FH12-40S-0.5SH_1x40-1MP_P0.50mm_Horizontal -> Connector_FFC-FPC:Hirose_FH12-40S-0.5SH_1x40-1MP_P0.50mm_Horizontal
- J4, J5: footprint Tag-Connect_TC2030-IDC-NL_2x03_P1.27mm_Vertical -> Connector:Tag-Connect_TC2030-IDC-NL_2x03_P1.27mm_Vertical
- LS1: footprint SpeakerPads_2.6mm -> OpenCycle:SpeakerPads_2.6mm
- Q1, Q2: footprint SOT-23 -> Package_TO_SOT_SMD:SOT-23
- R1, R10, R11, R12, R13, R14, R15, R16, R17, R18, R19, R2, R20, R21, R22, R23, R24, R25, R3, R4, R9: footprint R_0402_1005Metric -> Resistor_SMD:R_0402_1005Metric
- R5, R6, R7, R8: footprint R_0603_1608Metric -> Resistor_SMD:R_0603_1608Metric
- SW1, SW2, SW3: footprint SW_SPST_PTS810 -> Button_Switch_SMD:SW_SPST_PTS810
- SW4, SW5: footprint SW_Push_1P1T-MP_NO_Horizontal_Alps_SKRTLAE010 -> Button_Switch_SMD:SW_Push_1P1T-MP_NO_Horizontal_Alps_SKRTLAE010
- U1: footprint ESP32-S3-WROOM-1 -> RF_Module:ESP32-S3-WROOM-1
- U2: footprint Laird_BL652 -> RF_Module:Laird_BL652
- U3: footprint ublox_MAX -> RF_GPS:ublox_MAX
- U4: footprint Lite-On_LTR-303ALS-01 -> OptoDevice:Lite-On_LTR-303ALS-01
- U5: footprint SOT-223-3_TabPin2 -> Package_TO_SOT_SMD:SOT-223-3_TabPin2
- U6: footprint SOT-23-5 -> Package_TO_SOT_SMD:SOT-23-5
- U7: footprint TQFN-16-1EP_3x3mm_P0.5mm_EP1.23x1.23mm -> Package_DFN_QFN:TQFN-16-1EP_3x3mm_P0.5mm_EP1.23x1.23mm
- U8: footprint Bosch_LGA-10_2x2mm_P0.5mm_BMP581 -> OpenCycle:Bosch_LGA-10_2x2mm_P0.5mm_BMP581
Routing:
- net VBAT: track 0.00 -> 1.25 mm, vias 0 -> 1
- net I2C_SDA: track 0.00 -> 1.25 mm, vias 0 -> 1
- net I2C_SCL: track 0.00 -> 1.25 mm, vias 0 -> 1
